File: saleae_current_sensor.kicad_pcb (KiCad board)
At the start: 4 copper layers, 64 x 40.4 mm, 44 parts, among them J1 USB4505-03-0-A_REVA, J2 TSM-104-02-T-DH, M1 MountingHole_Pad, M2 MountingHole_Pad, M3 MountingHole_Pad, U1 TES_1-0523, U2 L78L12, U3 L7912, U4 ACS723xLCTR-05AB, U5 ACS723xLCTR-40AB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

Commit message: Misc updates kibuzzard lock in mounting holes/connectors change dielectric thickness for total 1.6mm stackup
Parts:
- added kibuzzard-64A244C5: G***, kibuzzard-64A244C5, F.Cu at (197.5, 133.2)
- added kibuzzard-64A244FA: G***, kibuzzard-64A244FA, F.Cu at (202.0, 119.4)
- added kibuzzard-64A24521: G***, kibuzzard-64A24521, F.Cu at (202.0, 147.4)
- added kibuzzard-64A24575: G***, kibuzzard-64A24575, F.Cu at (199.4, 133.5)
- moved M1 0.85 mm to (198.0, 113.0)
- moved M2 0.55 mm to (254.0, 113.0)
Other:
- board text removed: "HIGH VOLTAGE"
- board text removed: "POS CURRENT +-40A MAX"
